File: HypoV Breakout/HypoV Breakout.kicad_pcb (KiCad board)
At the start: 2 copper layers, 42 x 17.5 mm, 8 parts, among them J1 Conn_01x05_Pin, J3 Conn_01x05_Pin, U1 MAX30205, U2 MAX30205

Commit message: added final pcb
Parts:
- removed .1UF_C: C, Capacitor_SMD:C_0805_2012Metric_Pad1.18x1.45mm_HandSolder
- removed 4.7K_R, 4.7K_R2, 4.7K_R3: R, Resistor_SMD:R_0805_2012Metric_Pad1.20x1.40mm_HandSolder
- removed U1, U2: MAX30205, footprints:21-0137_T833&plus_2_MXM-M
Connections:
- J1 pad 1: +3V32 -> unconnected-(J1-Pin_1-Pad1)
- J1 pad 2: Net-(J1-Pin_2) -> unconnected-(J1-Pin_2-Pad2)
- J1 pad 3: Net-(J1-Pin_3) -> unconnected-(J1-Pin_3-Pad3)
- J1 pad 4: Net-(J1-Pin_4) -> unconnected-(J1-Pin_4-Pad4)
- J1 pad 5: GND2 -> unconnected-(J1-Pin_5-Pad5)
- J3 pad 1: +3V3 -> unconnected-(J3-Pin_1-Pad1)
- J3 pad 2: Net-(J3-Pin_2) -> unconnected-(J3-Pin_2-Pad2)
- J3 pad 3: Net-(J3-Pin_3) -> unconnected-(J3-Pin_3-Pad3)
- J3 pad 4: Net-(J3-Pin_4) -> unconnected-(J3-Pin_4-Pad4)
- J3 pad 5: GND -> unconnected-(J3-Pin_5-Pad5)
Routing:
- net +3V3: track 31.8 -> 0.00 mm
- net GND: track 20.5 -> 0.00 mm
- net GND2: track 16.7 -> 0.00 mm
- net Net-(J3-Pin_4): track 14.9 -> 0.00 mm
- net Net-(J3-Pin_3): track 12.5 -> 0.00 mm
- net +3V32: track 10.9 -> 0.00 mm
- net Net-(J3-Pin_2): track 9.36 -> 0.00 mm
- net Net-(J1-Pin_2): track 5.48 -> 0.00 mm
- net Net-(J1-Pin_4): track 5.31 -> 0.00 mm
- net Net-(J1-Pin_3): track 4.10 -> 0.00 mm
- added copper zone on F.Cu, net unconnected-(J1-Pin_5-Pad5)
- added copper zone on F.Cu, net unconnected-(J3-Pin_5-Pad5)
- removed copper zone on F.Cu, net GND
- removed copper zone on F.Cu, net GND2
