File: HypoV Breakout/HypoV Breakout.kicad_sch (KiCad schematic)
At the start: 8 parts, among them J1 Conn_01x05_Pin, J3 Conn_01x05_Pin, U1 MAX30205MTA+T, U2 MAX30205MTA+T

Commit message: added final pcb
Parts:
- removed C1: C, Capacitor_SMD:C_0805_2012Metric_Pad1.18x1.45mm_HandSolder, symbol Device:C
- removed R1, R2, R3: R, Resistor_SMD:R_0805_2012Metric_Pad1.20x1.40mm_HandSolder, symbol Device:R
- removed U1, U2: MAX30205MTA+T, footprints:21-0137_T833&plus_2_MXM-M, symbol hypo_temp_sensor:MAX30205MTA+T
Connections:
- net +3V3: no longer names the net of J3.1 (Pin_1)
- net +3V32: no longer names the net of J1.1 (Pin_1)
- net GND: no longer names the net of J3.5 (Pin_5)
- net GND2: no longer names the net of J1.5 (Pin_5)
